File: Design/HF0R0.brd (EAGLE design)
At the start: 34.6 x 90 mm, 6 parts, among them J1 3-644456-2, P1 HEXABIT_X3_ROW

Commit message: -The final design, all done.
Parts:
- removed P1: HEXABIT_X3_ROW, hexabitz_connectors:HEXABIT_X3_ROW
- added C1: 4.7uF, HEXABITZ_RCLS:C-0805
- added C2: 1uF, HEXABITZ_RCLS:C-0805
- added JP4, JP5: (no value), HEXABITZ_CONNECTION_PARTS:1X03
- added P2: HEXABIT_X3_ROW_NO_P7_P14, hexabitz_connectors:HEXABIT_X3_ROW_NO_P7_P14
- added R1: 1k, HEXABITZ_RCLS:R-0603
- added R2: 2k, HEXABITZ_RCLS:R-0603
- added U1: LDK130C33R, HEXABITZ_ICs:SOT65P210X110-5N
- JP3: device HEXABITZ_USER_INTERFACE_PARTS:1X01 -> HEXABITZ_CONNECTION_PARTS:1X03
- moved JP3 15.3 mm to (7.94, 39.1), turned to 180 degrees
- moved J1 13.0 mm to (-5.24, 38.7)
Connections:
- new net ARDUINO_RX0: JP1.1, JP5.2
- new net ARDUINO_TX0: JP1.2, R1.2
- new net GND: C1.2, C2.2, J1.1, JP2.7, P2.PAD_PD15, P2.PAD_PD16, P2.PAD_PD17, P2.PAD_PD18, P2.PAD_PD19, P2.PAD_PD20, P2.PAD_PD21, P2.PAD_PD22, P2.PAD_PD23, P2.PAD_PD24, P2.PAD_PD25, P2.PAD_PD26, P2.PAD_PD27, P2.PAD_PD28, R2.1, U1.2
- new net N$4: C2.1, J1.2, U1.1, U1.3
- new net PORT_12D: JP4.1, P2.PAD_PD12
- new net PORT_12U: JP5.1, P2.PAD_PU12
- new net PORT_1D: P2.PAD_PD1, P2.PAD_PD13
- new net PORT_1U: P2.PAD_PU1, P2.PAD_PU13
- new net PORT_2D: JP4.3, P2.PAD_PD2
- new net PORT_2U: JP5.3, P2.PAD_PU2
- new net PORT_3D: P2.PAD_PD11, P2.PAD_PD3
- new net PORT_3U: P2.PAD_PU11, P2.PAD_PU3
- new net PORT_4D: P2.PAD_PD10, P2.PAD_PD4
- new net PORT_4U: P2.PAD_PU10, P2.PAD_PU4
- new net PORT_5D: P2.PAD_PD5, P2.PAD_PD9
- new net PORT_5U: P2.PAD_PU5, P2.PAD_PU9
- new net PORT_6D: P2.PAD_PD6, P2.PAD_PD8
- new net PORT_6U: P2.PAD_PU6, P2.PAD_PU8
- new net VDD: JP3.2, P2.PAD_PU15, P2.PAD_PU16, P2.PAD_PU17, P2.PAD_PU18, P2.PAD_PU19, P2.PAD_PU20, P2.PAD_PU21, P2.PAD_PU22, P2.PAD_PU23, P2.PAD_PU24, P2.PAD_PU25, P2.PAD_PU26, P2.PAD_PU27, P2.PAD_PU28
- net N$1: now also C1.1, JP3.1, U1.5; no longer P1.PAD_PU15, P1.PAD_PU16, P1.PAD_PU17, P1.PAD_PU18, P1.PAD_PU19, P1.PAD_PU20, P1.PAD_PU21, P1.PAD_PU22, P1.PAD_PU23, P1.PAD_PU24, P1.PAD_PU25, P1.PAD_PU26, P1.PAD_PU27, P1.PAD_PU28
- net N$2: now also JP4.2, R1.1, R2.2; no longer P1.PAD_PD15, P1.PAD_PD16, P1.PAD_PD17, P1.PAD_PD18, P1.PAD_PD19, P1.PAD_PD20, P1.PAD_PD21, P1.PAD_PD22, P1.PAD_PD23, P1.PAD_PD24, P1.PAD_PD25, P1.PAD_PD26, P1.PAD_PD27, P1.PAD_PD28
Routing:
- net GND: track 0.00 -> 75.0 mm, vias 0 -> 12
- net VDD: track 0.00 -> 69.4 mm, vias 0 -> 4
- net ARDUINO_RX0: track 0.00 -> 51.0 mm
- net N$2: track 0.00 -> 43.0 mm
- net PORT_3U: track 0.00 -> 26.4 mm
- net PORT_4D: track 0.00 -> 26.2 mm, vias 0 -> 2
- net PORT_3D: track 0.00 -> 25.9 mm, vias 0 -> 2
- net PORT_4U: track 0.00 -> 25.5 mm
- net PORT_6D: track 0.00 -> 25.4 mm
- net PORT_5U: track 0.00 -> 25.3 mm, vias 0 -> 2
- net PORT_1U: track 0.00 -> 25.1 mm, vias 0 -> 2
- net PORT_1D: track 0.00 -> 25.1 mm
- net PORT_6U: track 0.00 -> 24.9 mm, vias 0 -> 2
- net PORT_5D: track 0.00 -> 24.8 mm
- net N$4: track 0.00 -> 14.8 mm, vias 0 -> 1
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- added copper zone on layer 16, net GND
- added copper zone on layer 16, net N$1
- added copper zone on layer 16, net N$4
- added copper zone on layer 1, net VDD
Other:
- board text added: "0"
- board text added: "1"
- board text added: "13"
- board text added: "2"
- board text added: "3"
- board text added: "3V3"
- board text added: "5V"
- board text added: "7"
- board text added: "8"
- board text added: "Ardo RX"
- board text added: "Ardo TX"
- board text added: "EXT"
- board text added: "GND"
- board text added: "HF0R00"
- board text added: "INT"
- board text added: "P1"
- board text added: "P2"
- board text added: "P3"
- board text added: "P4"
- board text added: "P5"
- board text added: "P6"
- board text added: "PWR_SEL"
