File: Design/HF0R0.sch (EAGLE design)
At the start: 6 parts, among them J1 3-644456-2, P1 HEXABIT_X3_ROW

Commit message: -The final design, all done.
Parts:
- removed P1: HEXABIT_X3_ROW, hexabitz_connectors:HEXABIT_X3_ROW
- added C1: 4.7uF, HEXABITZ_RCLS:C-0805
- added C2: 1uF, HEXABITZ_RCLS:C-0805
- added JP4, JP5: (no value), HEXABITZ_CONNECTION_PARTS:PINHD-1X3
- added P2: HEXABIT_X3_ROW_NO_P7_P14, hexabitz_connectors:HEXABIT_X3_ROW_NO_P7_P14
- added R1: 1k, HEXABITZ_RCLS:R-0603
- added R2: 2k, HEXABITZ_RCLS:R-0603
- added U1: LDK130C33R, HEXABITZ_ICs:LDK130C33R
- JP3: device HEXABITZ_USER_INTERFACE_PARTS:PINHD-1X1 -> HEXABITZ_CONNECTION_PARTS:PINHD-1X3
Connections:
- new net ARDUINO_RX0: JP1.1, JP5.2
- new net ARDUINO_TX0: JP1.2, R1.2
- new net GND: C1.2, C2.2, J1.1, JP2.7, P2.GND1, P2.GND10, P2.GND11, P2.GND12, P2.GND13, P2.GND14, P2.GND2, P2.GND3, P2.GND4, P2.GND5, P2.GND6, P2.GND7, P2.GND8, P2.GND9, R2.1, U1.GND
- new net N$4: C2.1, J1.2, U1.EN, U1.IN
- new net PORT_12D: JP4.1, P2.SD12
- new net PORT_12U: JP5.1, P2.SU12
- new net PORT_1D: P2.SD1, P2.SD13
- new net PORT_1U: P2.SU1, P2.SU13
- new net PORT_2D: JP4.3, P2.SD2
- new net PORT_2U: JP5.3, P2.SU2
- new net PORT_3D: P2.SD11, P2.SD3
- new net PORT_3U: P2.SU11, P2.SU3
- new net PORT_4D: P2.SD10, P2.SD4
- new net PORT_4U: P2.SU10, P2.SU4
- new net PORT_5D: P2.SD5, P2.SD9
- new net PORT_5U: P2.SU5, P2.SU9
- new net PORT_6D: P2.SD6, P2.SD8
- new net PORT_6U: P2.SU6, P2.SU8
- new net VDD: JP3.2, P2.VDD1, P2.VDD10, P2.VDD11, P2.VDD12, P2.VDD13, P2.VDD14, P2.VDD2, P2.VDD3, P2.VDD4, P2.VDD5, P2.VDD6, P2.VDD7, P2.VDD8, P2.VDD9
- net N$1: now also C1.1, JP3.1, U1.OUT; no longer P1.VDD1, P1.VDD10, P1.VDD11, P1.VDD12, P1.VDD13, P1.VDD14, P1.VDD2, P1.VDD3, P1.VDD4, P1.VDD5, P1.VDD6, P1.VDD7, P1.VDD8, P1.VDD9
- net N$2: now also JP4.2, R1.1, R2.2; no longer P1.GND1, P1.GND10, P1.GND11, P1.GND12, P1.GND13, P1.GND14, P1.GND2, P1.GND3, P1.GND4, P1.GND5, P1.GND6, P1.GND7, P1.GND8, P1.GND9
Other:
- note added: "0"
- moved on the sheet: J1, JP1, JP2
